Commit message: Simplified wheel and and added colision model

File: proxima_description/urdf/proxima_base.urdf.xacro (robot description, xacro)
@@ -3,4 +3,5 @@
   <!-- Mesh filenames -->
   <xacro:property name="mesh_platform" value="package://proxima_description/meshes/proxima/platform.stl"/>
+  <xacro:property name="mesh_platform_collision" value="package://proxima_description/meshes/proxima/platform_collision.stl"/>
   <xacro:property name="mesh_fork" value="package://proxima_description/meshes/proxima/fork.stl"/>
   <xacro:property name="mesh_wheel" value="package://proxima_description/meshes/proxima/wheel.stl"/>
@@ -23,5 +24,5 @@
       <origin xyz="0 0 0" rpy="0 0 0"/>
       <geometry>
-        <box size="0.3 0.7 0.25"/>
+        <mesh filename="${mesh_platform_collision}" scale="1 1 1"/>
       </geometry>
     </collision>
@@ -57,5 +58,5 @@
         <origin xyz="0 0 0" rpy="0 0 0"/>
         <geometry>
-          <mesh filename="${mesh_wheel}" scale="1 1 1"/>
+          <cylinder radius="0.12" length="0.12"/>
         </geometry>
         <material name="proxima_color"/>
@@ -64,5 +65,5 @@
         <origin xyz="0 0 0" rpy="0 0 0"/>
         <geometry>
-          <mesh filename="${mesh_wheel}" scale="1 1 1"/>
+          <cylinder radius="0.12" length="0.12"/>
         </geometry>
       </collision>

Commit message: Changed joint name

File: proxima_description/urdf/proxima_base.urdf.xacro (robot description, xacro)
@@ -69,5 +69,5 @@
       </collision>
     </link>
-    <joint name="${prefix}_joint" type="revolute">
+    <joint name="${prefix}_swerve_joint" type="revolute">
       <parent link="platform_link"/>
       <child link="${prefix}_fork_link"/>
