Commit message: Fixed wrong manip orientation

File: proxima_description/urdf/manipulators/6DOF.urdf.xacro (robot description, xacro)
@@ -33,5 +33,5 @@
           <mesh filename="package://proxima_description/meshes/manipulators/6DOF/base_assy.STL" scale="0.001 0.001 0.001"/>
         </geometry>
-        <origin xyz="0.0 0.0 0.0" rpy="0.0 0.0 ${pi/2}"/>
+        <origin xyz="0.0 0.0 0.0" rpy="0.0 0.0 -${pi/2}"/>
         <material name="gray">
           <color rgba=".796 .824 .937 1"/>
@@ -83,5 +83,5 @@
       <limit lower="-1.58" upper="1.58" effort="1000.0" velocity="0.5"/>
       <!-- <origin xyz="0 0 0.0" rpy="0 -0.2881 0"/> -->
-      <origin xyz="0 0.02727 0.07" rpy="0 0 ${pi/2}"/>
+      <origin xyz="0 -0.02727 0.07" rpy="0 0 -${pi/2}"/>
     </joint>
     <link name="link_3">
@@ -109,5 +109,5 @@
       <parent link="link_2"/>
       <child link="link_3"/>
-      <axis xyz="1 0 0"/>
+      <axis xyz="-1 0 0"/>
       <limit lower="-1.58" upper="1.58" effort="1000.0" velocity="0.5"/>
       <origin xyz="0.04573 0 0.495" rpy="0 0 0"/>
@@ -197,5 +197,5 @@
       <limit lower="-3.14" upper="3.14" effort="1000.0" velocity="0.5"/>
     </joint>
-    <link name="gripper_left">
+    <link name="gripper_right">
       <visual>
         <geometry>
@@ -219,18 +219,12 @@
       </inertial>
     </link>
-    <!-- Jaw opening per side: 0 = jaws touching (closed), 0.0326 = fully open (65.2 mm gap).
-         The joint limits leave 2 mm of travel beyond that working range: in DART a jaw
-         pressed against an active limit (e.g. by gravity) gets stuck there. MoveIt keeps
-         to the working range (sirius_moveit_config/config/joint_limits.yaml).
-         Both jaws are driven independently (no <mimic>): gz_ros2_control's mimic loop
-         oscillates and drove the jaws into their limits. -->
-    <joint name="joint_gripper_left" type="prismatic">
-      <origin xyz="0 -0.0174 0.05" rpy="0 0 0"/>
-      <parent link="tcp_connector"/>
-      <child link="gripper_left"/>
-      <axis xyz="0 -1 0"/>
+    <joint name="joint_gripper_right" type="prismatic">
+      <origin xyz="0 -0.052 0.05" rpy="0 0 0"/>
+      <parent link="tcp_connector"/>
+      <child link="gripper_right"/>
+      <axis xyz="0 1 0"/>
       <limit lower="-0.002" upper="0.0346" effort="100.0" velocity="0.1"/>
     </joint>
-    <link name="gripper_right">
+    <link name="gripper_left">
       <visual>
         <geometry>
@@ -254,9 +248,9 @@
       </inertial>
     </link>
-    <joint name="joint_gripper_right" type="prismatic">
-      <origin xyz="0 0.0174 0.05" rpy="0 0 0"/>
-      <parent link="tcp_connector"/>
-      <child link="gripper_right"/>
-      <axis xyz="0 1 0"/>
+    <joint name="joint_gripper_left" type="prismatic">
+      <origin xyz="0 0.052 0.05" rpy="0 0 0"/>
+      <parent link="tcp_connector"/>
+      <child link="gripper_left"/>
+      <axis xyz="0 -1 0"/>
       <limit lower="-0.002" upper="0.0346" effort="100.0" velocity="0.1"/>
     </joint>

Commit message: Fixed joint axis

File: proxima_description/urdf/manipulators/6DOF.urdf.xacro (robot description, xacro)
@@ -80,5 +80,5 @@
       <parent link="link_1"/>
       <child link="link_2"/>
-      <axis xyz="1 0 0"/>
+      <axis xyz="-1 0 0"/>
       <limit lower="-1.58" upper="1.58" effort="1000.0" velocity="0.5"/>
       <!-- <origin xyz="0 0 0.0" rpy="0 -0.2881 0"/> -->
